File: LM317.kicad_pcb (KiCad board)
At the start: 2 copper layers, 13 parts, among them J1 Conn_01x02, J2 Conn_01x02, U1 LM317_TO-220

Commit message: PCB Pendiente
Parts:
- removed C1: 2200uF, Capacitor_THT:CP_Radial_D14.0mm_P7.50mm
- removed C2, C4: 100nF, Capacitor_THT:C_Disc_D7.5mm_W2.5mm_P5.00mm
- removed C3: 10uF, Capacitor_THT:CP_Radial_D7.5mm_P2.50mm
- removed D1: D_Bridge_+AA-, Diode_THT:Diode_Bridge_Vishay_KBL
- removed D2: LED, LED_THT:LED_D5.0mm
- removed D3: 1N4007, Diode_THT:D_DO-41_SOD81_P10.16mm_Horizontal
- removed J1, J2: Conn_01x02, TerminalBlock:TerminalBlock_bornier-2_P5.08mm
- removed R1: 2k, Resistor_THT:R_Axial_DIN0207_L6.3mm_D2.5mm_P10.16mm_Horizontal
- removed R2: 240, Resistor_THT:R_Axial_DIN0204_L3.6mm_D1.6mm_P7.62mm_Horizontal
- removed RV1: 5k, Potentiometer_THT:Potentiometer_Alps_RK163_Single_Horizontal
- removed U1: LM317_TO-220, Package_TO_SOT_THT:TO-220-3_Vertical
