File: LM317.kicad_pcb (KiCad board)
At the start: 2 copper layers, 0 parts

Commit message: PCB Completa con Voltimetro
Parts:
- added C1: 2200uF, Capacitor_THT:CP_Radial_D14.0mm_P7.50mm, F.Cu at (154.4, 98.6)
- added C2: 100nF, Capacitor_THT:C_Disc_D7.5mm_W2.5mm_P5.00mm, F.Cu at (164.1, 97.5)
- added C3: 10uF, Capacitor_THT:CP_Radial_D7.5mm_P2.50mm, F.Cu at (170.2, 97.0)
- added C4: 100nF, Capacitor_THT:C_Disc_D7.5mm_W2.5mm_P5.00mm, F.Cu at (175.8, 98.0)
- added D1: D_Bridge_+AA-, Diode_THT:Diode_Bridge_Vishay_KBL, F.Cu at (142.7, 100.6)
- added D2: LED, LED_THT:LED_D5.0mm, F.Cu at (150.9, 74.2)
- added D3: 1N4007, Diode_THT:D_DO-41_SOD81_P10.16mm_Horizontal, F.Cu at (142.7, 105.7)
- added J1: Conn_01x02, TerminalBlock:TerminalBlock_bornier-2_P5.08mm, F.Cu at (133.1, 95.5)
- added J2: Conn_01x02, TerminalBlock:TerminalBlock_bornier-2_P5.08mm, F.Cu at (181.9, 98.6)
- added J3: Conn_01x03, Connector_PinSocket_2.54mm:PinSocket_1x03_P2.54mm_Vertical, F.Cu at (181.6, 80.0)
- added R1: 2k, Resistor_THT:R_Axial_DIN0207_L6.3mm_D2.5mm_P15.24mm_Horizontal, F.Cu at (148.3, 80.0)
- added R2: 240, Resistor_THT:R_Axial_DIN0204_L3.6mm_D1.6mm_P7.62mm_Horizontal, F.Cu at (162.1, 102.1)
- added RV1: 5k, Potentiometer_THT:Potentiometer_Alps_RK163_Single_Horizontal, F.Cu at (169.7, 74.7)
- added U1: LM317_TO-220, Package_TO_SOT_THT:TO-220-3_Vertical, F.Cu at (164.6, 108.2)
Routing:
- net ENTRADA: track 0.00 -> 130.3 mm
- net SALIDA: track 0.00 -> 75.9 mm
- net Net-(R2-Pad2): track 0.00 -> 52.7 mm, vias 0 -> 2
- net Net-(D2-Pad2): track 0.00 -> 20.0 mm
- net Net-(D1-Pad3): track 0.00 -> 9.65 mm
- net Net-(D1-Pad2): track 0.00 -> 9.65 mm
- net GND: vias 0 -> 1
- net (no net): vias 0 -> 3
- added copper zone on B.Cu, net GND
Other:
- board outline added: 55 x 40 mm
